File: Hardware/ESP32_TouchDown_Rev1/ESP32_TouchDown.sch (KiCad schematic (older format))
At the start: 68 parts, among them J2 Conn_02x07_Odd_Even, J3 B2B-PH-SM4-TB(LF)(SN), J4 Stemma, J5 USB_C_Receptacle_USB2.0, Q1 S8050, Q2 S8050, Q3 DMG3415U-7, Q4 S8050, SW1 TS-1088R-02526, SW2 TS-1088R-02526, SW3 SK-3296S-01-L3, U1 CP2102N-A01-GQFN28, U3 AP2112K-3.3, U4 ESP32-WROOM-32D, U5 MCP73831-2-OT

Commit message: Revision 1
Update KICAD project.
Parts:
- JP1: value 3V3/GPIO -> GPIO/3V3
- R22: value 1K -> 3.3K
- SW3: value SK-3296S-01-L3 -> K3-1280S-F1
- renumbered F2 to F1
Connections:
- net GND: now also FPC1.17 (DB0), FPC1.18 (DB1), FPC1.19 (DB2), FPC1.20 (DB3), FPC1.21 (DB4), FPC1.22 (DB5), FPC1.23 (DB6), FPC1.25 (DB8), FPC1.26 (DB9), FPC1.27 (DB10), FPC1.28 (DB11), FPC1.29 (DB12), FPC1.30 (DB13), FPC1.31 (DB14)
Other:
- note added: "C319148"
- note added: "C92658"
- note removed: "C319019"
Changed lines of the file:
@@
 P 7600 1800
 F 0 "SW3" H 7350 2300 50  0000 C CNN
-F 1 "SK-3296S-01-L3 " H 7350 2200 50  0000 C CNN
+F 1 "K3-1280S-F1 " H 7350 2200 50  0000 C CNN
 F 2 "Button_Switch_SMD:SW_SPDT_CK-JS102011SAQN" H 7600 1800 50  0001 C CNN
 F 3 "~" H 7600 1800 50  0001 C CNN
@@
 Text Notes 7700 2750 0    50   ~ 0
 ESP32 WROOM
-$Comp
-L ESP32_TouchDown:FPC_40P_0.5mm FPC1
-U 1 1 5F8810B4
-P 9800 4850
-F 0 "FPC1" H 9700 6850 50  0000 C CNN
-F 1 "FPC_40P_0.5mm" H 10200 2750 50  0000 C CNN
-F 2 "Connector_FFC-FPC:Hirose_FH12-40S-0.5SH_1x40-1MP_P0.50mm_Horizontal" H 10000 6050 50  0001 C CNN
-F 3 "" H 10000 6050 50  0001 C CNN
-	1    9800 4850
-	1    0    0    -1
-$EndComp
 Wire Notes Line
 	8400 2650 11150 2650
@@
 Wire Notes Line
 	11150 7200 8400 7200
-Connection ~ 9900 5300
 $Comp
 L power:GND #PWR0124
@@
 	1    0    0    -1
 $EndComp
-Wire Wire Line
-	10300 5300 9900 5300
 $Comp
 L power:GND #PWR0125
@@
 	1    0    0    -1
 $EndComp
-Wire Wire Line
-	10650 6800 9900 6800
 Wire Wire Line
 	10300 5350 10300 5300
@@
 $EndComp
 Wire Wire Line
-	10450 3600 9900 3600
-Wire Wire Line
 	9900 3500 9900 3600
 NoConn ~ 9900 3700
@@
 	1    0    0    -1
 $EndComp
-Wire Wire Line
-	10450 4100 9900 4100
 NoConn ~ 9900 4300
 Wire Wire Line
@@
 Wire Wire Line
 	10000 3900 9900 3900
-Wire Wire Line
-	10200 3400 9900 3400
 Text Notes 10500 2750 0    50   ~ 0
 TFT FPC 40 Pin
@@
 Text Notes 4850 1050 0    50   Italic 0
 C96616
-Text Notes 5000 2000 0    50   Italic 0
+Text Notes 5050 2000 0    50   Italic 0
 C51118
-Text Notes 7150 1550 0    50   Italic 0
-C319019
+Text Notes 7450 1550 0    50   Italic 0
+C92658
 Text Notes 11100 1600 1    50   Italic 0
 C160352
@@
 Text GLabel 10000 6300 2    50   Input ~ 0
 LED_K1
-Wire Wire Line
-	10250 6600 9900 6600
 Text GLabel 10000 6400 2    50   Input ~ 0
 LED_K2
@@
 	1    0    0    -1
 $EndComp
-Wire Wire Line
-	10650 6200 9900 6200
 Text GLabel 6400 6800 1    50   Input ~ 0
 TFT_LED
@@
 P 6700 6900
 F 0 "JP1" H 6700 7105 50  0000 C CNN
-F 1 "3V3/GPIO" H 6700 7014 50  0000 C CNN
+F 1 "GPIO/3V3" H 6700 7014 50  0000 C CNN
 F 2 "Jumper:SolderJumper-3_P1.3mm_Open_RoundedPad1.0x1.5mm_NumberLabels" H 6700 6900 50  0001 C CNN
 F 3 "~" H 6700 6900 50  0001 C CNN
@@
 P 6600 1750
 F 0 "R22" V 6500 1700 50  0000 L CNN
-F 1 "1K" V 6700 1700 50  0000 L CNN
+F 1 "3.3K" V 6700 1700 50  0000 L CNN
 F 2 "Resistor_SMD:R_0603_1608Metric" V 6530 1750 50  0001 C CNN
 F 3 "~" H 6600 1750 50  0001 C CNN
@@
 Connection ~ 2450 1150
 $Comp
-L Device:Polyfuse F2
+L Device:Polyfuse F1
 U 1 1 5FE0369E
 P 1950 850
-F 0 "F2" V 1725 850 50  0000 C CNN
+F 0 "F1" V 1725 850 50  0000 C CNN
 F 1 "Polyfuse" V 1816 850 50  0000 C CNN
 F 2 "Fuse:Fuse_0805_2012Metric" H 2000 650 50  0001 L CNN
@@
 	7900 1500 7900 1700
 Wire Wire Line
-	9900 4500 9900 5300
-Wire Wire Line
-	9900 5300 9900 6100
+	10650 6800 9900 6800
+Wire Wire Line
+	10250 6600 9900 6600
+Wire Wire Line
+	10650 6200 9900 6200
+Wire Wire Line
+	10450 4100 9900 4100
+Wire Wire Line
+	10450 3600 9900 3600
+Wire Wire Line
+	10200 3400 9900 3400
+Wire Wire Line
+	10300 5300 9900 5300
+$Comp
+L ESP32_TouchDown:FPC_40P_0.5mm FPC1
+U 1 1 5F8810B4
+P 9800 4850
+F 0 "FPC1" H 9700 6850 50  0000 C CNN
+F 1 "FPC_40P_0.5mm" H 10200 2750 50  0000 C CNN
+F 2 "Connector_FFC-FPC:Hirose_FH12-40S-0.5SH_1x40-1MP_P0.50mm_Horizontal" H 10000 6050 50  0001 C CNN
+F 3 "" H 10000 6050 50  0001 C CNN
+	1    9800 4850
+	1    0    0    -1
+$EndComp
+Wire Wire Line
+	9900 6100 9900 6000
+Wire Wire Line
+	9900 5900 9900 6000
+Connection ~ 9900 6000
+Wire Wire Line
+	9900 5900 9900 5800
+Connection ~ 9900 5900
+Wire Wire Line
+	9900 5800 9900 5700
+Connection ~ 9900 5800
+Wire Wire Line
+	9900 5700 9900 5600
+Connection ~ 9900 5700
+Connection ~ 9900 5300
+Connection ~ 9900 5400
+Wire Wire Line
+	9900 5400 9900 5300
+Connection ~ 9900 5500
+Wire Wire Line
+	9900 5500 9900 5400
+Connection ~ 9900 5600
+Wire Wire Line
+	9900 5600 9900 5500
+Wire Wire Line
+	9900 4500 9900 4600
+Connection ~ 9900 4600
+Wire Wire Line
+	9900 4600 9900 4700
+Connection ~ 9900 4700
+Wire Wire Line
+	9900 4700 9900 4800
+Connection ~ 9900 4800
+Wire Wire Line
+	9900 4800 9900 4900
+Connection ~ 9900 4900
+Wire Wire Line
+	9900 4900 9900 5000
+Connection ~ 9900 5000
+Wire Wire Line
+	9900 5000 9900 5100
+Connection ~ 9900 5100
+Wire Wire Line
+	9900 5100 9900 5200
+Connection ~ 9900 5200
+Wire Wire Line
+	9900 5200 9900 5300
+Text Notes 1350 2250 0    50   Italic 0
+C319148
 $EndSCHEMATC
